File: midicontrol.brd (EAGLE design)
At the start: 160 x 100 mm, 50 parts, among them CON1 B3B-ZR, J3 MABP 5S, U1 6N138S(TB), U3 74HC595D, U4 ATMEGA328P-AN

Commit message: nearly finished
Parts:
- removed 4DIG_7SEG1: (no value), 7-seg-disp:4DIG_7SEG
- removed CON1: B3B-ZR, jst:B3B-ZR
- removed J3: MABP 5S, MAB_5_SH:MAB-5-SH
- removed LIDAR_MOTOR, LIDAR_MOTOR1, LIDAR_MOTOR2, LIDAR_MOTOR3, LIDAR_MOTOR4, LIDAR_MOTOR5: JST-PH_2-PIN_HEADER, srg:JST_B2B-PH_HEADER
- removed RGB_LED: JST-PH_4-PIN_HEADER, srg:JST_B4B-PH_HEADER
- added BTN0, BTN1, BTN2, BTN3, BTN4, BTN5, PWR_IN: JST-PH_2-PIN_HEADER, srg:JST_B2B-PH_HEADER
- added C10, C11, C12, C13, C14, C9: 100nf, rcl:C1206
- added D1: BAT60JFILM, BAT60JFILM:SOD2513X117N
- added DIS1: NFD-5641BS, display-misc:NFD-5641
- added EXP: B3B-ZR, jst:B3B-ZR
- added IC1: FT232RL-TUBE, FT232RL-TUBE:SSOP28-LD
- added J1: UJ2-MIBH2-4-SMT-TR, UJ2-MIBH2-4-SMT-TR:CUI_UJ2-MIBH2-4-SMT-TR
- added PC2: 47u, rcl:PANASONIC_D
- added R19: 1M, SmartPrj:R0603-ROUND
- added R20: 27R, SmartPrj:R0603-ROUND
- added R21: 1k5, rcl:R0603
- added R22, R24: 22r, rcl:R0603
- added R23, R29: 1k, rcl:R0603
- added R25: 100r, rcl:R0603
- added R34: 100k, rcl:R0603
- added R35: 69k, rcl:R0603
- added S1: ESP201, olli:ESP201
- added SJ2: (no value), jumper:SJ
- added SW1: EC12E_SW, switch-alps:ALPS_EC12E_SW
- added Y2: 16MHz, SmartPrj:RESONATOR
- moved R18 372.0 mm to (61.0, 21.6), turned to 90 degrees
- moved R17 357.1 mm to (49.5, 21.6), turned to 90 degrees
- moved R16 342.2 mm to (38.1, 21.6), turned to 90 degrees
- moved R15 327.5 mm to (26.7, 21.6), turned to 90 degrees
- moved MIDI_IN 325.8 mm to (90.2, 85.1), flipped to the bottom, turned to 180 degrees
- moved R14 312.9 mm to (15.2, 21.6), turned to 90 degrees
- moved MIDI_OUT 287.7 mm to (39.4, 85.1), flipped to the bottom, turned to 180 degrees
- moved LED1 283.7 mm to (66.0, 87.6)
- moved U4 270.0 mm to (48.3, 67.3)
- moved U1 209.0 mm to (35.6, 73.7), turned to 180 degrees
- moved PCA9533 177.1 mm to (57.1, 90.2)
- moved ISP 155.4 mm to (92.7, 6.35), turned to 270 degrees
- moved CN1 142.0 mm to (5.08, 100.3), flipped to the bottom, turned to 180 degrees
- moved U3 113.4 mm to (58.4, 40.6)
Connections:
- removed net N$27: U4.22
- new net 3V3OUT: IC1.17
- new net BAT_LVL: R34.1, R35.2, U4.22
- new net D1: DIS1.P$6, U4.12
- new net D2: DIS1.P$8, U4.13
- new net D3: DIS1.P$9, U4.23
- new net D4: DIS1.P$12, U4.24
- new net N$25: IC1.5, R29.2
- new net N$28: J1.3, R21.1, R24.2
- new net N$29: C9.2, IC1.2
- new net N$30: D1.2, J1.1
- new net N$32: R25.1, SJ2.2
- new net N$34: J1.2, R22.2
- new net N$38: IC1.16, R22.1
- new net N$39: IC1.15, R24.1
- new net N$40: J1.SH1, J1.SH2, J1.SH3, J1.SH4, J1.SH5, R25.2
- new net XT1: R19.1, R20.2, Y2.3
- new net XTAL2: R19.2, U4.8, Y2.1
- net +5V: now also BTN0.P2, BTN1.P2, BTN2.P2, BTN3.P2, BTN4.P2, BTN5.P2, C11.2, C12.2, C13.1, C14.1, D1.1, EXP.1, IC1.20, IC1.4, PC2.+, R21.2, SW1.D; no longer CON1.1, LIDAR_MOTOR.P2, LIDAR_MOTOR1.P2, LIDAR_MOTOR2.P2, LIDAR_MOTOR3.P2, LIDAR_MOTOR4.P2, LIDAR_MOTOR5.P2
- net B0: now also BTN0.P1; no longer LIDAR_MOTOR.P1
- net B1: now also BTN1.P1; no longer LIDAR_MOTOR1.P1
- net B2: now also BTN2.P1; no longer LIDAR_MOTOR2.P1
- net B3: now also BTN3.P1, U4.25; no longer LIDAR_MOTOR3.P1, U4.24
- net B4: now also BTN4.P1, U4.26; no longer LIDAR_MOTOR4.P1, U4.25
- net B5: now also BTN5.P1; no longer LIDAR_MOTOR5.P1, U4.26
- net ENC_A: now also SW1.B
- net ENC_B: now also SW1.A
- net ENC_SW: now also SW1.E
- net EXP_IN: now also EXP.2, U4.19; no longer CON1.2, U4.23
- net GND: now also C10.2, C11.1, C12.1, C13.2, C14.2, EXP.3, IC1.18, IC1.21, IC1.25, IC1.26, IC1.7, J1.5, PC2.-, PWR_IN.P1, R35.1, SJ2.1, SW1.C, Y2.2; no longer CON1.3
- net MIDI_IN: now also R23.1
- net MIDI_OUT: now also R29.1
- net N$1: now also DIS1.P$11; no longer 4DIG_7SEG1.13
- net N$16: now also R20.1
- net N$19: now also IC1.1, R23.2; no longer U4.8
- net N$2: now also DIS1.P$7; no longer 4DIG_7SEG1.9
- net N$21: now also C10.1
- net N$26: now also C3.2, IC4.1, S1.P$1; no longer U4.19
- net N$3: now also DIS1.P$4; no longer 4DIG_7SEG1.4
- net N$4: now also DIS1.P$2; no longer 4DIG_7SEG1.2
- net N$5: now also DIS1.P$1; no longer 4DIG_7SEG1.1
- net N$6: now also DIS1.P$10; no longer 4DIG_7SEG1.12
- net N$7: now also DIS1.P$5; no longer 4DIG_7SEG1.5
- net N$8: now also DIS1.P$3; no longer 4DIG_7SEG1.3
- net PWR: now also PWR_IN.P2, R34.2, S1.P$3; no longer C3.2, IC4.1, IC4.3
- net RST: now also C9.1
